File: Power Sense 3.0/Power Sense 3.0.sch (KiCad schematic (older format))
At the start: 43 parts, among them IC1 MCP3909, J1 Power, J2 ProgHead, J3 SPI, T1 AC1030, T2 Murata_782485_55C, U1 PIC18F25K20_I/SS, Y1 3.579545MHz Crystal

Commit message: Updated files with new files
Changed lines of the file:
@@
 Text Label 6300 3050 0    60   ~ 0
 SDO
-Text Label 10100 2400 0    60   ~ 0
+Text Label 10100 3200 0    60   ~ 0
 SDI
 $Comp
@@
 L R R18
 U 1 1 5AB08AF1
-P 9950 2400
-F 0 "R18" V 9900 2250 50  0000 C CNN
-F 1 "1k" V 9950 2400 50  0000 C CNN
-F 2 "Resistors_THT:R_Axial_DIN0204_L3.6mm_D1.6mm_P7.62mm_Horizontal" V 9880 2400 50  0001 C CNN
-F 3 "" H 9950 2400 50  0001 C CNN
-	1    9950 2400
+P 9950 3200
+F 0 "R18" V 9900 3050 50  0000 C CNN
+F 1 "1k" V 9950 3200 50  0000 C CNN
+F 2 "Resistors_THT:R_Axial_DIN0204_L3.6mm_D1.6mm_P7.62mm_Horizontal" V 9880 3200 50  0001 C CNN
+F 3 "" H 9950 3200 50  0001 C CNN
+	1    9950 3200
 	0    1    1    0
 $EndComp
@@
 Text Label 6250 3450 0    60   ~ 0
 GND
-NoConn ~ 9700 3200
-Wire Wire Line
-	9700 2400 9800 2400
+Wire Wire Line
+	9700 3200 9800 3200
 NoConn ~ 6600 5500
 $Comp
@@
 NoConn ~ 1450 4750
 NoConn ~ 2250 4750
+NoConn ~ 9700 2400
 $EndSCHEMATC

Commit message: Load Cap Change
Change load capacitors from 30 pF to 27 pF
Parts:
- C8, C9: value 30pF -> 27pF
Changed lines of the file:
@@
 LIBS:valves
 LIBS:microchip_pic18mcu
-LIBS:symbols
 LIBS:mylib
 LIBS:Power Sense 3.0-cache
@@
 P 7350 3450
 F 0 "C9" H 7375 3550 50  0000 L CNN
-F 1 "30pF" V 7200 3450 50  0000 L CNN
+F 1 "27pF" V 7200 3450 50  0000 L CNN
 F 2 "Capacitors_THT:C_Disc_D3.0mm_W1.6mm_P2.50mm" H 7388 3300 50  0001 C CNN
 F 3 "" H 7350 3450 50  0001 C CNN
@@
 P 7350 3150
 F 0 "C8" H 7375 3250 50  0000 L CNN
-F 1 "30pF" V 7500 3150 50  0000 L CNN
+F 1 "27pF" V 7500 3150 50  0000 L CNN
 F 2 "Capacitors_THT:C_Disc_D3.0mm_W1.6mm_P2.50mm" H 7388 3000 50  0001 C CNN
 F 3 "" H 7350 3150 50  0001 C CNN

Commit message: Initial commit
- Created new branch for 3.1.
- Remapped symbols to schematic.
- Deleted CH1 circuitry
- Removed resistor from MCLR since it was removed during breadboard prototyping
Parts:
- removed R1: 150k 1W, Resistors_THT:R_Axial_DIN0414_L11.9mm_D4.5mm_P15.24mm_Horizontal, symbol R
- removed R20: 1k, Resistors_THT:R_Axial_DIN0204_L3.6mm_D1.6mm_P7.62mm_Horizontal, symbol R
- removed R4, R5: 200 1%, Resistors_THT:R_Axial_DIN0204_L3.6mm_D1.6mm_P7.62mm_Horizontal, symbol R
- removed T2: Murata_782485_55C, EMMS_FP:Murata_782485_Series, symbol Murata_782485_55C
- C1, C10, C2, C3, C4, C5, C6, C7, C8, C9: symbol C -> Device:C
- D1, D2, D3: symbol LED -> Device:LED
- IC1: symbol MCP3909 -> Power-Sense-3.0-rescue:MCP3909
- J1: symbol Conn_01x02_Male -> Power-Sense-3.0-rescue:Conn_01x02_Male
- J2: symbol Conn_01x05_Male -> Power-Sense-3.0-rescue:Conn_01x05_Male
- J3: symbol Conn_01x07_Male -> Power-Sense-3.0-rescue:Conn_01x07_Male
- R10, R11, R13, R14, R15, R16, R17, R18, R19, R2, R21, R22, R23, R3, R6, R7, R8, R9: symbol R -> Device:R
- T1: symbol AC1030 -> Power-Sense-3.0-rescue:AC1030
- U1: symbol PIC18F25K20_I/SS -> Power-Sense-3.0-rescue:PIC18F25K20_I_SS
- Y1: symbol Crystal -> Device:Crystal
Connections:
- wire segments 122 -> 131
- no-connect marks 12 -> 10

Commit message: Added transformer for CH1
Put new transformer sch symbol
Parts:
- added T?: Transformer_1P_1S, symbol Device:Transformer_1P_1S
Changed lines of the file:
@@
 Wire Wire Line
 	9700 3400 10100 3400
+$Comp
+L Device:Transformer_1P_1S T?
+U 1 1 5C003099
+P 1750 4750
+F 0 "T?" H 1750 5128 50  0000 C CNN
+F 1 "Transformer_1P_1S" H 1750 5037 50  0000 C CNN
+F 2 "" H 1750 4750 50  0001 C CNN
+F 3 "~" H 1750 4750 50  0001 C CNN
+	1    1750 4750
+	1    0    0    -1
+$EndComp
 $EndSCHEMATC

Commit message: Added new CH1 circuitry
Added transformer circuitry and resistor divider for CH1 of MCP
Parts:
- added R?: 536k, symbol Device:R
- added R?: 10k 1%, symbol Device:R
- added R? (x2): 1k, symbol Device:R
Connections:
- wire segments 131 -> 156
Changed lines of the file:
@@
 L power:GND #PWR01
 U 1 1 5AB00A66
-P 1050 5650
-F 0 "#PWR01" H 1050 5400 50  0001 C CNN
-F 1 "GND" H 1050 5500 50  0000 C CNN
-F 2 "" H 1050 5650 50  0001 C CNN
-F 3 "" H 1050 5650 50  0001 C CNN
-	1    1050 5650
-	1    0    0    -1
-$EndComp
-Text Label 1050 5600 0    60   ~ 0
+P 1050 6250
+F 0 "#PWR01" H 1050 6000 50  0001 C CNN
+F 1 "GND" H 1050 6100 50  0000 C CNN
+F 2 "" H 1050 6250 50  0001 C CNN
+F 3 "" H 1050 6250 50  0001 C CNN
+	1    1050 6250
+	1    0    0    -1
+$EndComp
+Text Label 1050 6200 0    60   ~ 0
 GND
 $Comp
@@
 	1    0    0    -1
 $EndComp
-Text Label 1050 4550 0    60   ~ 0
+Text Label 1000 4250 0    60   ~ 0
 H
-Text Label 1050 4950 0    60   ~ 0
+Text Label 1000 4650 0    60   ~ 0
 N
 $Comp
@@
 L Device:R R9
 U 1 1 5AB02FDE
-P 2950 5050
-F 0 "R9" V 3030 5050 50  0000 C CNN
-F 1 "1k" V 2950 5050 50  0000 C CNN
-F 2 "Resistors_THT:R_Axial_DIN0204_L3.6mm_D1.6mm_P7.62mm_Horizontal" V 2880 5050 50  0001 C CNN
-F 3 "" H 2950 5050 50  0001 C CNN
-	1    2950 5050
+P 2950 4750
+F 0 "R9" V 3030 4750 50  0000 C CNN
+F 1 "1k" V 2950 4750 50  0000 C CNN
+F 2 "Resistors_THT:R_Axial_DIN0204_L3.6mm_D1.6mm_P7.62mm_Horizontal" V 2880 4750 50  0001 C CNN
+F 3 "" H 2950 4750 50  0001 C CNN
+	1    2950 4750
 	0    -1   -1   0
 $EndComp
@@
 L Device:C C4
 U 1 1 5AB030D7
-P 3200 5200
-F 0 "C4" H 3225 5300 50  0000 L CNN
-F 1 "100nF" H 3300 5200 50  0000 L CNN
-F 2 "Capacitors_THT:C_Disc_D3.0mm_W1.6mm_P2.50mm" H 3238 5050 50  0001 C CNN
-F 3 "" H 3200 5200 50  0001 C CNN
-	1    3200 5200
+P 3200 4900
+F 0 "C4" H 3225 5000 50  0000 L CNN
+F 1 "100nF" H 3300 4900 50  0000 L CNN
+F 2 "Capacitors_THT:C_Disc_D3.0mm_W1.6mm_P2.50mm" H 3238 4750 50  0001 C CNN
+F 3 "" H 3200 4900 50  0001 C CNN
+	1    3200 4900
 	1    0    0    -1
 $EndComp
@@
 Text Label 3200 4050 0    60   ~ 0
 GND
-Text Label 3200 5350 0    60   ~ 0
+Text Label 3200 5050 0    60   ~ 0
 GND
 Text Label 3200 2600 0    60   ~ 0
@@
 L Power-Sense-3.0-rescue:Conn_01x02_Male J1
 U 1 1 5AB1B19B
-P 1650 5850
-F 0 "J1" H 1650 5950 50  0000 C CNN
-F 1 "Power" H 1650 5650 50  0000 C CNN
-F 2 "Pin_Headers:Pin_Header_Straight_1x02_Pitch2.54mm" H 1650 5850 50  0001 C CNN
-F 3 "" H 1650 5850 50  0001 C CNN
-	1    1650 5850
-	0    -1   -1   0
-$EndComp
-Text Label 1650 5450 0    60   ~ 0
+P 1650 6450
+F 0 "J1" H 1650 6550 50  0000 C CNN
+F 1 "Power" H 1650 6250 50  0000 C CNN
+F 2 "Pin_Headers:Pin_Header_Straight_1x02_Pitch2.54mm" H 1650 6450 50  0001 C CNN
+F 3 "" H 1650 6450 50  0001 C CNN
+	1    1650 6450
+	0    -1   -1   0
+$EndComp
+Text Label 1650 6050 0    60   ~ 0
 H
-Text Label 1750 5450 0    60   ~ 0
+Text Label 1750 6050 0    60   ~ 0
 N
 $Comp
@@
 L Device:LED D1
 U 1 1 5AB2D6B3
-P 2800 5700
-F 0 "D1" H 2800 5800 50  0000 C CNN
-F 1 "LED" H 2800 5600 50  0000 C CNN
-F 2 "LEDs:LED_D5.0mm" H 2800 5700 50  0001 C CNN
-F 3 "" H 2800 5700 50  0001 C CNN
-	1    2800 5700
-	1    0    0    -1
-$EndComp
-Text Label 2450 5700 2    60   ~ 0
+P 2800 5750
+F 0 "D1" H 2800 5850 50  0000 C CNN
+F 1 "LED" H 2800 5650 50  0000 C CNN
+F 2 "LEDs:LED_D5.0mm" H 2800 5750 50  0001 C CNN
+F 3 "" H 2800 5750 50  0001 C CNN
+	1    2800 5750
+	1    0    0    -1
+$EndComp
+Text Label 2450 5750 2    60   ~ 0
 GND
 $Comp
 L Device:R R10
 U 1 1 5AB2E835
-P 3200 5700
-F 0 "R10" V 3280 5700 50  0000 C CNN
-F 1 "330" V 3200 5700 50  0000 C CNN
-F 2 "Resistors_THT:R_Axial_DIN0204_L3.6mm_D1.6mm_P7.62mm_Horizontal" V 3130 5700 50  0001 C CNN
-F 3 "" H 3200 5700 50  0001 C CNN
-	1    3200 5700
-	0    -1   -1   0
-$EndComp
-Text Label 3500 5700 0    60   ~ 0
+P 3200 5750
+F 0 "R10" V 3280 5750 50  0000 C CNN
+F 1 "330" V 3200 5750 50  0000 C CNN
+F 2 "Resistors_THT:R_Axial_DIN0204_L3.6mm_D1.6mm_P7.62mm_Horizontal" V 3130 5750 50  0001 C CNN
+F 3 "" H 3200 5750 50  0001 C CNN
+	1    3200 5750
+	0    -1   -1   0
+$EndComp
+Text Label 3500 5750 0    60   ~ 0
 LED_TO_25
 Text Label 9900 2300 0    60   ~ 0
@@
 NoConn ~ 9700 3000
 Wire Wire Line
-	1050 5650 1050 5450
+	1050 6250 1050 6050
 Wire Wire Line
 	4150 2650 4800 2650
@@
 	3200 3150 4800 3150
 Wire Wire Line
-	1150 4550 1050 4550
-Wire Wire Line
 	3100 4450 3200 4450
 Wire Wire Line
-	3100 5050 3200 5050
-Wire Wire Line
-	3650 3250 4800 3250
+	3100 4750 3200 4750
+Wire Wire Line
+	3650 3250 3750 3250
 Wire Wire Line
 	3650 4450 3650 3250
 Wire Wire Line
 	3750 3350 4800 3350
-Wire Wire Line
-	3750 5050 3750 3350
-Connection ~ 3200 5050
+Connection ~ 3200 4750
 Connection ~ 3200 4450
 Wire Wire Line
@@
 Connection ~ 7000 3450
 Wire Wire Line
-	1650 5650 1650 5450
-Wire Wire Line
-	1750 5650 1750 5450
+	1650 6250 1650 6050
+Wire Wire Line
+	1750 6250 1750 6050
 Wire Wire Line
 	4650 5500 4650 5300
@@
 Connection ~ 8800 3800
 Wire Wire Line
-	2950 5700 3050 5700
-Wire Wire Line
-	2650 5700 2450 5700
+	2950 5750 3050 5750
+Wire Wire Line
+	2650 5750 2450 5750
 Wire Wire Line
 	9900 2300 9700 2300
 Wire Wire Line
-	3500 5700 3350 5700
+	3500 5750 3350 5750
 Wire Wire Line
 	4150 2850 4800 2850
@@
 	2000 2900 2800 2900
 Wire Wire Line
-	3200 5050 3750 5050
+	3200 4750 3750 4750
 Wire Wire Line
 	3200 4450 3650 4450
@@
 	9750 2200 9900 2200
 Wire Wire Line
-	1050 4950 1150 4950
+	1000 4650 1100 4650
 Wire Wire Line
 	9700 3400 10100 3400
@@
 L Device:Transformer_1P_1S T?
 U 1 1 5C003099
-P 1750 4750
-F 0 "T?" H 1750 5128 50  0000 C CNN
-F 1 "Transformer_1P_1S" H 1750 5037 50  0000 C CNN
-F 2 "" H 1750 4750 50  0001 C CNN
-F 3 "~" H 1750 4750 50  0001 C CNN
-	1    1750 4750
-	1    0    0    -1
-$EndComp
+P 1600 4450
+F 0 "T?" H 1600 4828 50  0000 C CNN
+F 1 "Transformer_1P_1S" H 1600 4737 50  0000 C CNN
+F 2 "" H 1600 4450 50  0001 C CNN
+F 3 "~" H 1600 4450 50  0001 C CNN
+	1    1600 4450
+	1    0    0    -1
+$EndComp
+Wire Wire Line
+	1150 4250 1150 4750
+Wire Wire Line
+	1000 4250 1150 4250
+Wire Wire Line
+	1200 4250 1150 4250
+Connection ~ 1150 4250
+Wire Wire Line
+	1200 4650 1100 4650
+Connection ~ 1100 4650
+$Comp
+L Device:R R?
+U 1 1 5C01C71E
+P 1400 4900
+F 0 "R?" H 1330 4854 50  0000 R CNN
+F 1 "536k" H 1330 4945 50  0000 R CNN
+F 2 "" V 1330 4900 50  0001 C CNN
+F 3 "~" H 1400 4900 50  0001 C CNN
+	1    1400 4900
+	-1   0    0    1
+$EndComp
+$Comp
+L Device:R R?
+U 1 1 5C021CEE
+P 2150 4300
+F 0 "R?" H 2080 4254 50  0000 R CNN
+F 1 "10k 1%" H 2080 4345 50  0000 R CNN
+F 2 "" V 2080 4300 50  0001 C CNN
+F 3 "~" H 2150 4300 50  0001 C CNN
+	1    2150 4300
+	-1   0    0    1
+$EndComp
+$Comp
+L Device:R R?
+U 1 1 5C02248A
+P 2150 4600
+F 0 "R?" H 2080 4554 50  0000 R CNN
+F 1 "1k" H 2080 4645 50  0000 R CNN
+F 2 "" V 2080 4600 50  0001 C CNN
+F 3 "~" H 2150 4600 50  0001 C CNN
+	1    2150 4600
+	-1   0    0    1
+$EndComp
+Wire Wire Line
+	3750 4750 3750 3350
+Wire Wire Line
+	2000 4250 2000 4150
+Wire Wire Line
+	2000 4150 2150 4150
+Connection ~ 3750 3250
+Wire Wire Line
+	3750 3250 4800 3250
+Connection ~ 3750 3350
+Wire Wire Line
+	3750 3350 3750 3250
+Wire Wire Line
+	2150 4500 2150 4450
+Connection ~ 2150 4450
+Wire Wire Line
+	2000 4650 2000 4750
+Wire Wire Line
+	2000 4750 2150 4750
+$Comp
+L Device:R R?
+U 1 1 5C06402E
+P 1400 5200
+F 0 "R?" H 1330 5154 50  0000 R CNN
+F 1 "1k" H 1330 5245 50  0000 R CNN
+F 2 "" V 1330 5200 50  0001 C CNN
+F 3 "~" H 1400 5200 50  0001 C CNN
+	1    1400 5200
+	-1   0    0    1
+$EndComp
+Wire Wire Line
+	1100 5350 1400 5350
+Wire Wire Line
+	1100 4650 1100 5350
+Wire Wire Line
+	1150 4750 1400 4750
+Wire Wire Line
+	1400 5050 2550 5050
+Connection ~ 1400 5050
+Wire Wire Line
+	1400 5350 1750 5350
+Wire Wire Line
+	1750 5350 1750 5150
+Wire Wire Line
+	1750 5150 2650 5150
+Connection ~ 1400 5350
+Wire Wire Line
+	1400 5350 1400 5450
+Wire Wire Line
+	2150 4750 2150 4850
+Connection ~ 2150 4750
+Text Label 1400 5450 0    60   ~ 0
+GND
+Text Label 2150 4850 0    60   ~ 0
+GND
+Wire Wire Line
+	2150 4450 2550 4450
+Wire Wire Line
+	2550 5050 2550 4450
+Connection ~ 2550 4450
+Wire Wire Line
+	2550 4450 2800 4450
+Wire Wire Line
+	2650 5150 2650 4750
+Wire Wire Line
+	2150 4750 2650 4750
+Connection ~ 2650 4750
+Wire Wire Line
+	2650 4750 2800 4750
 $EndSCHEMATC

Commit message: Updated schematic for Power Sense
Updated schematic for Power Sense to include new transformer and resistor divider components.

**Incomplete PCB Layout**
Parts:
- R1, R12, R4, R5: renamed from R?; footprint (none) -> Resistor_THT:R_Axial_DIN0204_L3.6mm_D1.6mm_P7.62mm_Horizontal
- T2: renamed from T?; footprint (none) -> EMMS_FP:Transformer FS12-090-C2
Connections:
- wire segments 156 -> 157
Changed lines of the file:
@@
 	-1   0    0    1
 $EndComp
-Text Label 4150 1850 0    60   ~ 0
-+5V
 Text Label 4600 2400 2    60   ~ 0
 GND
@@
 	1050 6250 1050 6050
 Wire Wire Line
-	4150 2650 4800 2650
-Wire Wire Line
 	4150 2250 4150 2400
 Connection ~ 4150 2400
@@
 Wire Wire Line
 	3500 5750 3350 5750
-Wire Wire Line
-	4150 2850 4800 2850
-Connection ~ 4150 2650
 Wire Wire Line
 	4800 2750 4150 2750
@@
 	9700 3400 10100 3400
 $Comp
-L Device:Transformer_1P_1S T?
+L Device:Transformer_1P_1S T2
 U 1 1 5C003099
 P 1600 4450
-F 0 "T?" H 1600 4828 50  0000 C CNN
+F 0 "T2" H 1600 4828 50  0000 C CNN
 F 1 "Transformer_1P_1S" H 1600 4737 50  0000 C CNN
-F 2 "" H 1600 4450 50  0001 C CNN
+F 2 "EMMS_FP:Transformer FS12-090-C2" H 1600 4450 50  0001 C CNN
 F 3 "~" H 1600 4450 50  0001 C CNN
 	1    1600 4450
@@
 Connection ~ 1100 4650
 $Comp
-L Device:R R?
+L Device:R R1
 U 1 1 5C01C71E
 P 1400 4900
-F 0 "R?" H 1330 4854 50  0000 R CNN
+F 0 "R1" H 1330 4854 50  0000 R CNN
 F 1 "536k" H 1330 4945 50  0000 R CNN
-F 2 "" V 1330 4900 50  0001 C CNN
+F 2 "Resistor_THT:R_Axial_DIN0204_L3.6mm_D1.6mm_P7.62mm_Horizontal" V 1330 4900 50  0001 C CNN
 F 3 "~" H 1400 4900 50  0001 C CNN
 	1    1400 4900
@@
 $EndComp
 $Comp
-L Device:R R?
+L Device:R R5
 U 1 1 5C021CEE
 P 2150 4300
-F 0 "R?" H 2080 4254 50  0000 R CNN
+F 0 "R5" H 2080 4254 50  0000 R CNN
 F 1 "10k 1%" H 2080 4345 50  0000 R CNN
-F 2 "" V 2080 4300 50  0001 C CNN
+F 2 "Resistor_THT:R_Axial_DIN0204_L3.6mm_D1.6mm_P7.62mm_Horizontal" V 2080 4300 50  0001 C CNN
 F 3 "~" H 2150 4300 50  0001 C CNN
 	1    2150 4300
@@
 $EndComp
 $Comp
-L Device:R R?
+L Device:R R12
 U 1 1 5C02248A
 P 2150 4600
-F 0 "R?" H 2080 4554 50  0000 R CNN
+F 0 "R12" H 2080 4554 50  0000 R CNN
 F 1 "1k" H 2080 4645 50  0000 R CNN
-F 2 "" V 2080 4600 50  0001 C CNN
+F 2 "Resistor_THT:R_Axial_DIN0204_L3.6mm_D1.6mm_P7.62mm_Horizontal" V 2080 4600 50  0001 C CNN
 F 3 "~" H 2150 4600 50  0001 C CNN
 	1    2150 4600
@@
 	2000 4750 2150 4750
 $Comp
-L Device:R R?
+L Device:R R4
 U 1 1 5C06402E
 P 1400 5200
-F 0 "R?" H 1330 5154 50  0000 R CNN
+F 0 "R4" H 1330 5154 50  0000 R CNN
 F 1 "1k" H 1330 5245 50  0000 R CNN
-F 2 "" V 1330 5200 50  0001 C CNN
+F 2 "Resistor_THT:R_Axial_DIN0204_L3.6mm_D1.6mm_P7.62mm_Horizontal" V 1330 5200 50  0001 C CNN
 F 3 "~" H 1400 5200 50  0001 C CNN
 	1    1400 5200
@@
 Wire Wire Line
 	2650 4750 2800 4750
+$Comp
+L power:PWR_FLAG #FLG0101
+U 1 1 5C02E13C
+P 750 6250
+F 0 "#FLG0101" H 750 6325 50  0001 C CNN
+F 1 "PWR_FLAG" H 750 6423 50  0000 C CNN
+F 2 "" H 750 6250 50  0001 C CNN
+F 3 "~" H 750 6250 50  0001 C CNN
+	1    750  6250
+	-1   0    0    1
+$EndComp
+Wire Wire Line
+	750  6250 750  6050
+Wire Wire Line
+	4150 2850 4800 2850
+Wire Wire Line
+	4150 2650 4800 2650
+Connection ~ 4150 2650
+Text Label 750  6200 0    60   ~ 0
++5V
+Text Label 4150 1900 0    60   ~ 0
++5V
 $EndSCHEMATC

Commit message: Finished Version of initial v3.1
Added connections to all new parts and added silkscreen components
Parts:
- removed T2: Transformer_1P_1S, EMMS_FP:Transformer FS12-090-C2, symbol Device:Transformer_1P_1S
- added J4: TestHeader, Connector_PinHeader_2.54mm:PinHeader_1x06_P2.54mm_Vertical, symbol Connector_Generic:Conn_01x06
- added R20, R24: 0, Resistor_THT:R_Axial_DIN0204_L3.6mm_D1.6mm_P7.62mm_Horizontal, symbol Device:R
- added T2: 2p2sTransformer, EMMS_FP:Transformer FS12-090-C2, symbol mylib:2p2sTransformer
- J3: footprint Pin_Headers:Pin_Header_Straight_1x07_Pitch2.54mm -> Connector_PinHeader_2.54mm:PinHeader_1x07_P2.54mm_Vertical
Connections:
- net labels added: CH0+, CH1+
- wire segments 157 -> 165
Changed lines of the file:
@@
 	1    0    0    -1
 $EndComp
-Text Label 1000 4250 0    60   ~ 0
+Text Label 950  4050 0    60   ~ 0
 H
-Text Label 1000 4650 0    60   ~ 0
+Text Label 950  4700 0    60   ~ 0
 N
 $Comp
@@
 F 0 "J3" H 6300 6100 50  0000 C CNN
 F 1 "SPI" V 6200 5700 50  0000 C CNN
-F 2 "Pin_Headers:Pin_Header_Straight_1x07_Pitch2.54mm" H 6300 5700 50  0001 C CNN
+F 2 "Connector_PinHeader_2.54mm:PinHeader_1x07_P2.54mm_Vertical" H 6300 5700 50  0001 C CNN
 F 3 "" H 6300 5700 50  0001 C CNN
 	1    6300 5700
@@
 	3100 4750 3200 4750
 Wire Wire Line
-	3650 3250 3750 3250
-Wire Wire Line
 	3650 4450 3650 3250
 Wire Wire Line
@@
 	9750 2200 9900 2200
 Wire Wire Line
-	1000 4650 1100 4650
+	950  4700 1050 4700
 Wire Wire Line
 	9700 3400 10100 3400
-$Comp
-L Device:Transformer_1P_1S T2
-U 1 1 5C003099
-P 1600 4450
-F 0 "T2" H 1600 4828 50  0000 C CNN
-F 1 "Transformer_1P_1S" H 1600 4737 50  0000 C CNN
-F 2 "EMMS_FP:Transformer FS12-090-C2" H 1600 4450 50  0001 C CNN
-F 3 "~" H 1600 4450 50  0001 C CNN
-	1    1600 4450
-	1    0    0    -1
-$EndComp
-Wire Wire Line
-	1150 4250 1150 4750
-Wire Wire Line
-	1000 4250 1150 4250
-Wire Wire Line
-	1200 4250 1150 4250
-Connection ~ 1150 4250
-Wire Wire Line
-	1200 4650 1100 4650
-Connection ~ 1100 4650
+Wire Wire Line
+	1450 4700 1050 4700
+Connection ~ 1050 4700
 $Comp
 L Device:R R1
 U 1 1 5C01C71E
-P 1400 4900
-F 0 "R1" H 1330 4854 50  0000 R CNN
-F 1 "536k" H 1330 4945 50  0000 R CNN
-F 2 "Resistor_THT:R_Axial_DIN0204_L3.6mm_D1.6mm_P7.62mm_Horizontal" V 1330 4900 50  0001 C CNN
-F 3 "~" H 1400 4900 50  0001 C CNN
-	1    1400 4900
+P 1600 4900
+F 0 "R1" H 1530 4854 50  0000 R CNN
+F 1 "536k" H 1530 4945 50  0000 R CNN
+F 2 "Resistor_THT:R_Axial_DIN0204_L3.6mm_D1.6mm_P7.62mm_Horizontal" V 1530 4900 50  0001 C CNN
+F 3 "~" H 1600 4900 50  0001 C CNN
+	1    1600 4900
 	-1   0    0    1
 $EndComp
@@
 	3750 4750 3750 3350
 Wire Wire Line
-	2000 4250 2000 4150
-Wire Wire Line
-	2000 4150 2150 4150
-Connection ~ 3750 3250
-Wire Wire Line
-	3750 3250 4800 3250
-Connection ~ 3750 3350
-Wire Wire Line
-	3750 3350 3750 3250
+	1850 4050 2150 4050
+Wire Wire Line
+	2150 4050 2150 4150
 Wire Wire Line
 	2150 4500 2150 4450
 Connection ~ 2150 4450
 Wire Wire Line
-	2000 4650 2000 4750
-Wire Wire Line
 	2000 4750 2150 4750
 $Comp
 L Device:R R4
 U 1 1 5C06402E
-P 1400 5200
-F 0 "R4" H 1330 5154 50  0000 R CNN
-F 1 "1k" H 1330 5245 50  0000 R CNN
-F 2 "Resistor_THT:R_Axial_DIN0204_L3.6mm_D1.6mm_P7.62mm_Horizontal" V 1330 5200 50  0001 C CNN
-F 3 "~" H 1400 5200 50  0001 C CNN
-	1    1400 5200
+P 1600 5200
+F 0 "R4" H 1530 5154 50  0000 R CNN
+F 1 "1k" H 1530 5245 50  0000 R CNN
+F 2 "Resistor_THT:R_Axial_DIN0204_L3.6mm_D1.6mm_P7.62mm_Horizontal" V 1530 5200 50  0001 C CNN
+F 3 "~" H 1600 5200 50  0001 C CNN
+	1    1600 5200
 	-1   0    0    1
 $EndComp
 Wire Wire Line
-	1100 5350 1400 5350
-Wire Wire Line
-	1100 4650 1100 5350
-Wire Wire Line
-	1150 4750 1400 4750
-Wire Wire Line
-	1400 5050 2550 5050
-Connection ~ 1400 5050
-Wire Wire Line
-	1400 5350 1750 5350
-Wire Wire Line
-	1750 5350 1750 5150
-Wire Wire Line
-	1750 5150 2650 5150
-Connection ~ 1400 5350
-Wire Wire Line
-	1400 5350 1400 5450
+	1050 4700 1050 5350
+Wire Wire Line
+	1800 5350 1800 5150
+Connection ~ 1600 5350
 Wire Wire Line
 	2150 4750 2150 4850
 Connection ~ 2150 4750
-Text Label 1400 5450 0    60   ~ 0
+Text Label 1600 5450 0    60   ~ 0
 GND
 Text Label 2150 4850 0    60   ~ 0
@@
 Text Label 4150 1900 0    60   ~ 0
 +5V
+$Comp
+L Connector_Generic:Conn_01x06 J4
+U 1 1 5C0294C7
+P 7950 5700
+F 0 "J4" H 8000 6050 50  0000 R CNN
+F 1 "TestHeader" V 8050 5800 50  0000 R CNN
+F 2 "Connector_PinHeader_2.54mm:PinHeader_1x06_P2.54mm_Vertical" H 7950 5700 50  0001 C CNN
+F 3 "~" H 7950 5700 50  0001 C CNN
+	1    7950 5700
+	0    -1   1    0
+$EndComp
+Wire Wire Line
+	7750 5500 7750 5300
+Wire Wire Line
+	7850 5500 7850 5300
+Wire Wire Line
+	7950 5500 7950 5300
+Wire Wire Line
+	8050 5500 8050 5300
+Wire Wire Line
+	8150 5500 8150 5300
+Wire Wire Line
+	8250 5500 8250 5300
+Text Label 8250 5300 1    60   ~ 0
+GND
+Text Label 7750 5300 1    60   ~ 0
+Fo0toPIC
+Text Label 7850 5300 1    60   ~ 0
+Fo1toPIC
+Text Label 7950 5300 1    60   ~ 0
+HFtoPIC
+Text Label 4400 3050 0    60   ~ 0
+CH0+
+Text Label 4400 3350 0    60   ~ 0
+CH1+
+Wire Wire Line
+	3650 3250 4800 3250
+$Comp
+L Device:R R24
+U 1 1 5C09C93D
+P 1300 5350
+F 0 "R24" V 1400 5350 50  0000 C CNN
+F 1 "0" V 1300 5350 50  0000 C CNN
+F 2 "Resistor_THT:R_Axial_DIN0204_L3.6mm_D1.6mm_P7.62mm_Horizontal" V 1230 5350 50  0001 C CNN
+F 3 "~" H 1300 5350 50  0001 C CNN
+	1    1300 5350
+	0    1    1    0
+$EndComp
+$Comp
+L Device:R R20
+U 1 1 5C0B30A6
+P 1300 4850
+F 0 "R20" V 1200 4850 50  0000 C CNN
+F 1 "0" V 1300 4850 50  0000 C CNN
+F 2 "Resistor_THT:R_Axial_DIN0204_L3.6mm_D1.6mm_P7.62mm_Horizontal" V 1230 4850 50  0001 C CNN
+F 3 "~" H 1300 4850 50  0001 C CNN
+	1    1300 4850
+	0    1    1    0
+$EndComp
+$Comp
+L mylib:2p2sTransformer T2
+U 1 1 5C0C4786
+P 2250 4000
+F 0 "T2" H 1650 4197 60  0000 C CNN
+F 1 "2p2sTransformer" H 1650 4091 60  0000 C CNN
+F 2 "EMMS_FP:Transformer FS12-090-C2" H 2250 4700 60  0001 C CNN
+F 3 "" H 2250 4700 60  0001 C CNN
+	1    2250 4000
+	1    0    0    -1
+$EndComp
+Wire Wire Line
+	950  4050 1150 4050
+Connection ~ 1150 4050
+Wire Wire Line
+	1150 4050 1450 4050
+Wire Wire Line
+	1450 4350 1450 4400
+Wire Wire Line
+	2000 4750 2000 4350
+Wire Wire Line
+	2000 4350 1850 4350
+Wire Wire Line
+	1800 5150 2650 5150
+Wire Wire Line
+	1600 5350 1800 5350
+Wire Wire Line
+	1600 5350 1600 5450
+Wire Wire Line
+	1150 4050 1150 4850
+Wire Wire Line
+	1050 5350 1150 5350
+Wire Wire Line
+	1450 5350 1600 5350
+Wire Wire Line
+	1450 4850 1450 4750
+Wire Wire Line
+	1450 4750 1600 4750
+Wire Wire Line
+	1600 5050 2550 5050
+Connection ~ 1600 5050
+Text Label 8150 5300 1    60   ~ 0
+CH0+
+Text Label 8050 5300 1    60   ~ 0
+CH1+
 $EndSCHEMATC

Commit message: First round of edits
Edited things in README.txt
See that file for changes
Connections:
- net labels added: CH1-
Changed lines of the file:
@@
 CH0+
 Text Label 8050 5300 1    60   ~ 0
-CH1+
+CH1-
+Text Label 4400 3250 0    60   ~ 0
+CH1-
 $EndSCHEMATC
