File: Power Sense 3.0/Power Sense 3.0.sch (KiCad schematic (older format))
At the start: 46 parts, among them IC1 MCP3909, J1 Power, J2 ProgHead, J3 SPI, J4 TestHeader, T1 AC1030, T2 2p2sTransformer, U1 PIC18F25K20_I/SS, Y1 3.579545MHz Crystal

Commit message: Changed Transformer Resistor Divider R value
Changed 10k to 20k for 240v use
Parts:
- R5: value 10k 1% -> 20k 1%
Changed lines of the file:
@@
 P 2150 4300
 F 0 "R5" H 2080 4254 50  0000 R CNN
-F 1 "10k 1%" H 2080 4345 50  0000 R CNN
+F 1 "20k 1%" H 2080 4345 50  0000 R CNN
 F 2 "Resistor_THT:R_Axial_DIN0204_L3.6mm_D1.6mm_P7.62mm_Horizontal" V 2080 4300 50  0001 C CNN
 F 3 "~" H 2150 4300 50  0001 C CNN

Commit message: 3.1.2
Removed two resistors in SCH and PCB
Fixed 5V connection on SPI connector
Parts:
- removed R15, R16: 10, Resistors_THT:R_Axial_DIN0204_L3.6mm_D1.6mm_P7.62mm_Horizontal, symbol Device:R
Connections:
- wire segments 165 -> 159
Changed lines of the file:
@@
 	6600 5500 6600 5300
 Wire Wire Line
-	9700 2200 9750 2200
-Wire Wire Line
 	8800 3700 8800 3800
 Wire Wire Line
@@
 Wire Wire Line
 	9700 1900 9900 1900
-Wire Wire Line
-	9700 2000 9850 2000
 Wire Wire Line
 	9700 2100 9900 2100
@@
 Wire Wire Line
 	9350 1600 9450 1600
-Wire Wire Line
-	9850 1500 9850 2000
-Connection ~ 9850 2000
-$Comp
-L Device:R R16
-U 1 1 5AB4153A
-P 9850 1350
-F 0 "R16" V 9750 1350 50  0000 C CNN
-F 1 "10" V 9850 1350 50  0000 C CNN
-F 2 "Resistors_THT:R_Axial_DIN0204_L3.6mm_D1.6mm_P7.62mm_Horizontal" V 9780 1350 50  0001 C CNN
-F 3 "" H 9850 1350 50  0001 C CNN
-	1    9850 1350
-	-1   0    0    1
-$EndComp
-Wire Wire Line
-	9850 1200 9850 1100
-Text Label 9850 1100 0    60   ~ 0
-+5V
-Wire Wire Line
-	9750 1650 9750 2200
-Connection ~ 9750 2200
 Wire Wire Line
 	6500 3150 7000 3150
@@
 NoConn ~ 6600 5500
 $Comp
-L Device:R R15
-U 1 1 5ABC818E
-P 9750 1500
-F 0 "R15" V 9650 1500 50  0000 C CNN
-F 1 "10" V 9750 1500 50  0000 C CNN
-F 2 "Resistors_THT:R_Axial_DIN0204_L3.6mm_D1.6mm_P7.62mm_Horizontal" V 9680 1500 50  0001 C CNN
-F 3 "" H 9750 1500 50  0001 C CNN
-	1    9750 1500
-	-1   0    0    1
-$EndComp
-Wire Wire Line
-	9750 1350 9750 1100
-Text Label 9750 1100 2    60   ~ 0
-+5V
-$Comp
 L Device:LED D2
 U 1 1 5ABCA984
@@
 Wire Wire Line
 	8800 1600 8800 1700
-Wire Wire Line
-	9850 2000 9900 2000
-Wire Wire Line
-	9750 2200 9900 2200
 Wire Wire Line
 	950  4700 1050 4700
@@
 Text Label 4400 3250 0    60   ~ 0
 CH1-
+Wire Wire Line
+	9700 2000 9900 2000
+Wire Wire Line
+	9700 2200 9900 2200
 $EndSCHEMATC
